File: tests/fixtures/test_03A_fixture.kicad_sch (KiCad schematic)
At the start: 3 parts, among them J1 Conn_01x02, SW1 Val, SW2 Val

Commit message: added updated tf 03A with footprint encodings
Parts:
- J1: footprint (none) -> |(5,5,0)S40
- SW1: footprint (none) -> |(5,5,0)R20
- SW2: footprint (none) -> |(5,6,0)R20
Changed lines of the file:
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@@
 			)
 		)
-		(property "Footprint" ""
+		(property "Footprint" "|(5,6,0)R20"
 			(at 119.38 102.362 0)
 			(effects
@@
 			)
 		)
-		(property "Footprint" ""
+		(property "Footprint" "|(5,5,0)R20"
 			(at 119.38 73.152 0)
 			(effects
@@
 			)
 		)
-		(property "Footprint" ""
+		(property "Footprint" "|(5,5,0)S40"
 			(at 153.67 86.36 0)
 			(effects
