File: tests/fixtures/test_03A_fixture.kicad_sch (KiCad schematic)
At the start: 3 parts, among them J1 Conn_01x02, SW1 Val, SW2 Val

Commit message: Migrate test fixtures from Footprint to LocLoad custom field
Move component location and electrical load encoding from overloaded
Footprint field to new custom LocLoad field. Remove leading pipe
character from encoding format.

Changes:
- Clear Footprint field values (restore to empty string)
- Add LocLoad custom property with format: (FS,WL,BL){S|L|R|G}<value>
- Remove leading | character from encoding format
- Add test_06 fixture files for new test cases

All fixtures now use LocLoad field as single source of component data.

🤖 Generated with [Claude Code](https://claude.com/claude-code)

Co-Authored-By: Claude <noreply@anthropic.com>
Parts:
- J1: footprint |(5,5,0)S40 -> (none); LocLoad (none) -> (5,5,0)S40
- SW1: footprint |(5,5,0)R20 -> (none); LocLoad (none) -> (5,5,0)R20
- SW2: footprint |(5,6,0)R20 -> (none); LocLoad (none) -> (5,6,0)R20
Changed lines of the file:
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@@
 			)
 		)
-		(property "Footprint" "|(5,6,0)R20"
+		(property "Footprint" ""
 			(at 119.38 102.362 0)
 			(effects
@@
 					(size 0.635 0.635)
 				)
+			)
+		)
+		(property "LocLoad" "(5,6,0)R20"
+			(at 119.38 105.41 0)
+			(effects
+				(font
+					(size 1.27 1.27)
+				)
+				(hide yes)
 			)
 		)
@@
 			)
 		)
-		(property "Footprint" "|(5,5,0)R20"
+		(property "Footprint" ""
 			(at 119.38 73.152 0)
 			(effects
@@
 					(size 0.635 0.635)
 				)
+			)
+		)
+		(property "LocLoad" "(5,5,0)R20"
+			(at 119.38 76.2 0)
+			(effects
+				(font
+					(size 1.27 1.27)
+				)
+				(hide yes)
 			)
 		)
@@
 			)
 		)
-		(property "Footprint" "|(5,5,0)S40"
+		(property "Footprint" ""
 			(at 153.67 86.36 0)
 			(effects
@@
 			(at 153.67 86.36 0)
 			(effects
+				(font
+					(size 1.27 1.27)
+				)
+				(hide yes)
+			)
+		)
+		(property "LocLoad" "(5,5,0)S40"
+			(at 153.67 86.36 0)
+			(effects
