File: tests/fixtures/test_02_fixture.kicad_sch (KiCad schematic)
At the start: 3 parts, among them SW1 Desc

Commit message: Migrate test fixtures from Footprint to LocLoad custom field
Move component location and electrical load encoding from overloaded
Footprint field to new custom LocLoad field. Remove leading pipe
character from encoding format.

Changes:
- Clear Footprint field values (restore to empty string)
- Add LocLoad custom property with format: (FS,WL,BL){S|L|R|G}<value>
- Remove leading | character from encoding format
- Add test_06 fixture files for new test cases

All fixtures now use LocLoad field as single source of component data.

🤖 Generated with [Claude Code](https://claude.com/claude-code)

Co-Authored-By: Claude <noreply@anthropic.com>
Parts:
- BT1: footprint |(10,0,0)S40 -> (none); LocLoad (none) -> (10,0,0)S40
- L1: footprint |(0,10,0)L2.1 -> (none); LocLoad (none) -> (0,10,0)L2.1
- SW1: footprint |(0,0,0)r20 -> (none); LocLoad (none) -> (0,0,0)r20
Changed lines of the file:
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@@
 			)
 		)
-		(property "Footprint" "|(10,0,0)S40"
+		(property "Footprint" ""
 			(at 115.57 75.946 90)
 			(effects
@@
 		)
 		(property "Description" "Multiple-cell battery"
+			(at 115.57 77.47 0)
+			(effects
+				(font
+					(size 1.27 1.27)
+				)
+				(hide yes)
+			)
+		)
+		(property "LocLoad" "(10,0,0)S40"
 			(at 115.57 77.47 0)
 			(effects
@@
 			)
 		)
-		(property "Footprint" "|(0,0,0)r20"
+		(property "Footprint" ""
 			(at 77.47 66.802 0)
 			(effects
@@
 					(size 0.635 0.635)
 				)
+			)
+		)
+		(property "LocLoad" "(0,0,0)r20"
+			(at 77.47 69.85 0)
+			(effects
+				(font
+					(size 1.27 1.27)
+				)
+				(hide yes)
 			)
 		)
@@
 			)
 		)
-		(property "Footprint" "|(0,10,0)L2.1"
+		(property "Footprint" ""
 			(at 104.14 52.07 90)
 			(effects
@@
 			)
 		)
+		(property "LocLoad" "(0,10,0)L2.1"
+			(at 104.14 52.07 0)
+			(effects
+				(font
+					(size 1.27 1.27)
+				)
+				(hide yes)
+			)
+		)
