File: tests/fixtures/test_04_fixture.kicad_sch (KiCad schematic)
At the start: 5 parts, among them SW1 Desc

Commit message: Migrate test fixtures from Footprint to LocLoad custom field
Move component location and electrical load encoding from overloaded
Footprint field to new custom LocLoad field. Remove leading pipe
character from encoding format.

Changes:
- Clear Footprint field values (restore to empty string)
- Add LocLoad custom property with format: (FS,WL,BL){S|L|R|G}<value>
- Remove leading | character from encoding format
- Add test_06 fixture files for new test cases

All fixtures now use LocLoad field as single source of component data.

🤖 Generated with [Claude Code](https://claude.com/claude-code)

Co-Authored-By: Claude <noreply@anthropic.com>
Parts:
- BT1: footprint |(0,0,0)S40 -> (none); LocLoad (none) -> (0,0,0)S40
- L1: footprint |(10,1,0)L1.5 -> (none); LocLoad (none) -> (10,1,0)L1.5
- L2: footprint |(10,2,0)L1.5 -> (none); LocLoad (none) -> (10,2,0)L1.5
- L3: footprint |(10,3,0)L1.5 -> (none); LocLoad (none) -> (10,3,0)L1.5
- SW1: footprint |(5,0,0)R20 -> (none); LocLoad (none) -> (5,0,0)R20
Changed lines of the file:
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@@
 			)
 		)
-		(property "Footprint" "|(0,0,0)S40"
+		(property "Footprint" ""
 			(at 151.13 91.186 90)
 			(effects
@@
 		)
 		(property "Description" "Single-cell battery"
+			(at 151.13 92.71 0)
+			(effects
+				(font
+					(size 1.27 1.27)
+				)
+				(hide yes)
+			)
+		)
+		(property "LocLoad" "(0,0,0)S40"
 			(at 151.13 92.71 0)
 			(effects
@@
 			)
 		)
-		(property "Footprint" "|(5,0,0)R20"
+		(property "Footprint" ""
 			(at 140.97 68.072 0)
 			(effects
@@
 					(size 0.635 0.635)
 				)
+			)
+		)
+		(property "LocLoad" "(5,0,0)R20"
+			(at 140.97 71.12 0)
+			(effects
+				(font
+					(size 1.27 1.27)
+				)
+				(hide yes)
 			)
 		)
@@
 			)
 		)
-		(property "Footprint" "|(10,2,0)L1.5"
+		(property "Footprint" ""
 			(at 113.03 64.77 90)
 			(effects
@@
 					(size 0.635 0.635)
 				)
+			)
+		)
+		(property "LocLoad" "(10,2,0)L1.5"
+			(at 113.03 64.77 0)
+			(effects
+				(font
+					(size 1.27 1.27)
+				)
+				(hide yes)
 			)
 		)
@@
 			)
 		)
-		(property "Footprint" "|(10,1,0)L1.5"
+		(property "Footprint" ""
 			(at 113.03 49.53 90)
 			(effects
@@
 					(size 0.635 0.635)
 				)
+			)
+		)
+		(property "LocLoad" "(10,1,0)L1.5"
+			(at 113.03 49.53 0)
+			(effects
+				(font
+					(size 1.27 1.27)
+				)
+				(hide yes)
 			)
 		)
@@
 			)
 		)
-		(property "Footprint" "|(10,3,0)L1.5"
+		(property "Footprint" ""
 			(at 113.03 80.01 90)
 			(effects
@@
 			)
 		)
+		(property "LocLoad" "(10,3,0)L1.5"
+			(at 113.03 80.01 0)
+			(effects
+				(font
+					(size 1.27 1.27)
+				)
+				(hide yes)
+			)
+		)
