File: tests/fixtures/test_05A_fixture.kicad_sch (KiCad schematic)
At the start: 6 parts, among them SW1 Desc

Commit message: Migrate test fixtures from Footprint to LocLoad custom field
Move component location and electrical load encoding from overloaded
Footprint field to new custom LocLoad field. Remove leading pipe
character from encoding format.

Changes:
- Clear Footprint field values (restore to empty string)
- Add LocLoad custom property with format: (FS,WL,BL){S|L|R|G}<value>
- Remove leading | character from encoding format
- Add test_06 fixture files for new test cases

All fixtures now use LocLoad field as single source of component data.

🤖 Generated with [Claude Code](https://claude.com/claude-code)

Co-Authored-By: Claude <noreply@anthropic.com>
Parts:
- BT1: footprint |(1,0,0)S40 -> (none); LocLoad (none) -> (1,0,0)S40
- FH1: footprint |(0,10,0)R50 -> (none); LocLoad (none) -> (0,10,0)R50
- GB1: footprint |(0,-10,0)R40 -> (none); LocLoad (none) -> (0,-10,0)R40
- L1: footprint |(0,0,100)L2.5 -> (none); LocLoad (none) -> (0,0,100)L2.5
- L2: footprint |(0,0,-100)L2.5 -> (none); LocLoad (none) -> (0,0,-100)L2.5
- SW1: footprint |(10,0,0)R20 -> (none); LocLoad (none) -> (10,0,0)R20
Changed lines of the file:
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@@
 			)
 		)
-		(property "Footprint" "|(1,0,0)S40"
+		(property "Footprint" ""
 			(at 68.58 64.516 90)
 			(effects
@@
 		)
 		(property "Description" "Single-cell battery"
+			(at 68.58 66.04 0)
+			(effects
+				(font
+					(size 1.27 1.27)
+				)
+				(hide yes)
+			)
+		)
+		(property "LocLoad" "(1,0,0)S40"
 			(at 68.58 66.04 0)
 			(effects
@@
 			)
 		)
-		(property "Footprint" "|(0,0,-100)L2.5"
+		(property "Footprint" ""
 			(at 187.96 57.15 90)
 			(effects
@@
 					(size 0.635 0.635)
 				)
+			)
+		)
+		(property "LocLoad" "(0,0,-100)L2.5"
+			(at 187.96 57.15 0)
+			(effects
+				(font
+					(size 1.27 1.27)
+				)
+				(hide yes)
 			)
 		)
@@
 			)
 		)
-		(property "Footprint" "|(0,0,100)L2.5"
+		(property "Footprint" ""
 			(at 186.69 39.37 90)
 			(effects
@@
 					(size 0.635 0.635)
 				)
+			)
+		)
+		(property "LocLoad" "(0,0,100)L2.5"
+			(at 186.69 39.37 0)
+			(effects
+				(font
+					(size 1.27 1.27)
+				)
+				(hide yes)
 			)
 		)
@@
 			)
 		)
-		(property "Footprint" "|(10,0,0)R20"
+		(property "Footprint" ""
 			(at 162.56 42.418 0)
 			(effects
@@
 					(size 0.635 0.635)
 				)
+			)
+		)
+		(property "LocLoad" "(10,0,0)R20"
+			(at 162.56 39.37 0)
+			(effects
+				(font
+					(size 1.27 1.27)
+				)
+				(hide yes)
 			)
 		)
@@
 			)
 		)
-		(property "Footprint" "|(0,10,0)R50"
+		(property "Footprint" ""
 			(at 102.87 53.34 0)
 			(effects
@@
 		(property "Description" ""
 			(at 102.87 53.34 0)
+			(effects
+				(font
+					(size 1.27 1.27)
+				)
+				(hide yes)
+			)
+		)
+		(property "LocLoad" "(0,10,0)R50"
+			(at 114.3 50.8 90)
 			(effects
 				(font
@@
 			)
 		)
-		(property "Footprint" "|(0,-10,0)R40"
+		(property "Footprint" ""
 			(at 102.87 80.01 0)
 			(effects
@@
 			(effects
 				(font
+					(size 1.27 1.27)
+				)
+				(hide yes)
+			)
+		)
+		(property "LocLoad" "(0,-10,0)R40"
+			(at 116.84 81.28 90)
+			(effects
+				(font
