File: tests/fixtures/test_08_fixture.kicad_sch (KiCad schematic)
At the start: 15 parts, among them SW1 Batt/Alt Master, SW2 Strobe, SW3 Nav Lght

Commit message: Add component value and description to component diagram titles
Component diagrams now display the component's value and description
in the title block, making it easy to identify what component the
diagram represents.

Changes:
- Updated generate_svg() to accept component_value and component_desc parameters
- Updated generate_component_diagrams() to look up and pass component info
- Added component info line in SVG title for component diagrams

SVG Title Format for Component Diagrams:
- Line 1: Project title - Rev X.X - Date (if title_block available)
- Line 2: CompRef: Value - Description (new!)
- Line 3: CompRef Component Diagram (bold)
- Line 4: Scale and coordinate info

Example:
  Simplified Z-11 - Rev 1.0 - 2025-10-26
  CB1: 30A - Circuit Breaker
  CB1 Component Diagram
  Scale: 8.5 px/inch | FS: 10"-50" | BL: 20"-40" (compressed)

System diagrams unchanged - still show system name.

All 265 tests passing.

🤖 Generated with [Claude Code](https://claude.com/claude-code)

Co-Authored-By: Claude <noreply@anthropic.com>
Connections:
- net P3B: now reaches B1.1 (Conn), SW1.4 (ON)
- net P3C: now reaches B1.2, LRU1.1 (Ylw), RG1.Val_A (F)
- net P3A: now reaches C1., FH1.1 (Pwr), R1.2, SW1.5 (IN)
- net at FH1.Val_A (Desc): now also SW2.2 (IN)
- net P1A: now reaches BT1.1 (+), C1.
- net P2A: now reaches C1., SW1.2 (IN)
- net L2A: now reaches L2.1 (In), L3.1 (In), SW3.1 (ON)
- net L1A: now reaches L1.1 (In), SW2.1 (ON)
- net P5A: now reaches RG1.Val_A (F)
- net P5A: now also A1. (OUTPUT)
- net P5B: now reaches A1. (OUTPUT)
- net P5B: now also R1.1 (Conn); no longer RG1.Val_A (F)
- net E1A: now reaches LRU2.1 (Ylw), R1.
- net E1B: now reaches LRU2.2 (Blk), R1.
Other:
- moved on the sheet: FH1
Changed lines of the file:
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@@
 	(wire
 		(pts
-			(xy 68.58 130.81) (xy 68.58 172.72)
-		)
-		(stroke
-			(width 0)
-			(type default)
-		)
-	)
-	(wire
-		(pts
-			(xy 74.93 124.46) (xy 74.93 148.59)
+			(xy 68.58 135.89) (xy 68.58 172.72)
+		)
+		(stroke
+			(width 0)
+			(type default)
+		)
+	)
+	(wire
+		(pts
+			(xy 74.93 129.54) (xy 74.93 148.59)
 		)
 		(stroke
@@
 	(wire
 		(pts
-			(xy 53.34 92.71) (xy 53.34 95.25)
+			(xy 53.34 92.71) (xy 53.34 100.33)
 		)
 		(stroke
@@
 	(wire
 		(pts
-			(xy 62.23 130.81) (xy 68.58 130.81)
-		)
-		(stroke
-			(width 0)
-			(type default)
-		)
-	)
-	(wire
-		(pts
-			(xy 62.23 124.46) (xy 74.93 124.46)
+			(xy 62.23 135.89) (xy 68.58 135.89)
+		)
+		(stroke
+			(width 0)
+			(type default)
+		)
+	)
+	(wire
+		(pts
+			(xy 62.23 129.54) (xy 74.93 129.54)
 		)
 		(stroke
@@
 			(width 0)
 			(type default)
+		)
+	)
+	(label "P4A"
+		(at 53.34 97.79 0)
+		(effects
+			(font
+				(size 1.27 1.27)
+			)
+			(justify left bottom)
+		)
+	)
+	(label "P3E"
+		(at 119.38 96.52 0)
+		(effects
+			(font
+				(size 1.27 1.27)
+			)
+			(justify left bottom)
+		)
+	)
+	(label "P2A"
+		(at 59.69 85.09 0)
+		(effects
+			(font
+				(size 1.27 1.27)
+			)
+			(justify left bottom)
+		)
+	)
+	(label "G6A"
+		(at 176.53 118.11 0)
+		(effects
+			(font
+				(size 1.27 1.27)
+			)
+			(justify left bottom)
+		)
+	)
+	(label "P5A"
+		(at 163.83 86.36 0)
+		(effects
+			(font
+				(size 1.27 1.27)
+			)
+			(justify left bottom)
+		)
+	)
+	(label "G1A"
+		(at 22.86 102.87 0)
+		(effects
+			(font
+				(size 1.27 1.27)
+			)
+			(justify left bottom)
+		)
+	)
+	(label "L1A"
+		(at 95.25 146.05 0)
+		(effects
+			(font
+				(size 1.27 1.27)
+			)
+			(justify left bottom)
+		)
+	)
+	(label "G2A"
+		(at 119.38 116.84 0)
+		(effects
+			(font
+				(size 1.27 1.27)
+			)
+			(justify left bottom)
+		)
+	)
+	(label "P5C"
+		(at 185.42 66.04 0)
+		(effects
+			(font
+				(size 1.27 1.27)
+			)
+			(justify left bottom)
+		)
+	)
+	(label "E1B"
+		(at 193.04 76.2 0)
+		(effects
+			(font
+				(size 1.27 1.27)
+			)
+			(justify left bottom)
+		)
+	)
+	(label "G5A"
+		(at 119.38 181.61 0)
+		(effects
+			(font
+				(size 1.27 1.27)
+			)
+			(justify left bottom)
+		)
+	)
+	(label "G4A"
+		(at 118.11 165.1 0)
+		(effects
+			(font
+				(size 1.27 1.27)
+			)
+			(justify left bottom)
+		)
+	)
+	(label "P3A"
+		(at 68.58 92.71 0)
+		(effects
+			(font
+				(size 1.27 1.27)
+			)
+			(justify left bottom)
+		)
+	)
+	(label "P5B"
+		(at 185.42 96.52 0)
+		(effects
+			(font
+				(size 1.27 1.27)
+			)
+			(justify left bottom)
+		)
+	)
+	(label "P1A"
+		(at 22.86 72.39 0)
+		(effects
+			(font
+				(size 1.27 1.27)
+			)
+			(justify left bottom)
+		)
+	)
+	(label "G3A"
+		(at 123.19 158.75 0)
+		(effects
+			(font
+				(size 1.27 1.27)
+			)
+			(justify left bottom)
+		)
+	)
+	(label "P2B"
+		(at 110.49 82.55 0)
+		(effects
+			(font
+				(size 1.27 1.27)
+			)
+			(justify left bottom)
+		)
+	)
+	(label "P3D"
+		(at 143.51 87.63 0)
+		(effects
+			(font
+				(size 1.27 1.27)
+			)
+			(justify left bottom)
+		)
+	)
+	(label "E1A"
+		(at 193.04 86.36 0)
+		(effects
+			(font
+				(size 1.27 1.27)
+			)
+			(justify left bottom)
+		)
+	)
+	(label "L2B"
+		(at 100.33 181.61 0)
+		(effects
+			(font
+				(size 1.27 1.27)
+			)
+			(justify left bottom)
+		)
+	)
+	(label "P3B"
+		(at 107.95 90.17 0)
+		(effects
+			(font
+				(size 1.27 1.27)
+			)
+			(justify left bottom)
+		)
+	)
+	(label "P3C"
+		(at 127 90.17 0)
+		(effects
+			(font
+				(size 1.27 1.27)
+			)
+			(justify left bottom)
+		)
+	)
+	(label "L2A"
+		(at 99.06 165.1 0)
+		(effects
+			(font
+				(size 1.27 1.27)
+			)
+			(justify left bottom)
 		)
 	)
@@
 	(symbol
 		(lib_id "AeroElectricConnectionSymbols:Fuse_Holder_6x")
-		(at 57.15 116.84 0)
+		(at 57.15 121.92 0)
 		(unit 1)
 		(exclude_from_sim no)
@@
 		(fields_autoplaced yes)
 		(property "Reference" "FH1"
-			(at 53.594 131.572 90)
+			(at 53.594 136.652 90)
 			(do_not_autoplace yes)
 			(effects
@@
 		)
 		(property "Value" "Panel Fuse Block"
-			(at 53.34 125.73 90)
+			(at 53.34 130.81 90)
 			(do_not_autoplace yes)
 			(effects
@@
 		)
 		(property "Footprint" ""
-			(at 54.61 105.41 0)
+			(at 54.61 110.49 0)
 			(effects
 				(font
@@
 		)
 		(property "Datasheet" ""
-			(at 54.61 105.41 0)
+			(at 54.61 110.49 0)
 			(effects
 				(font
@@
 		)
 		(property "Description" ""
-			(at 54.61 105.41 0)
+			(at 54.61 110.49 0)
 			(effects
 				(font
@@
 		)
 		(property "LocLoad" "(40,20,10)R40"
-			(at 57.15 116.84 90)
-			(effects
-				(font
+			(at 57.15 121.92 90)
+			(effects
+				(font

Commit message: Fix multipoint power symbol bug and add diagram enhancements
Bug Fixes:
- Fix multipoint connections with power symbols (GND, +12V, etc.)
  Power symbols now correctly treated as common pin in multipoint
  groups since all components connect to same global net
- Fix UnboundLocalError when components missing LocLoad data
  Wire length calculation now handles missing component coordinates
  gracefully with fallback to default length
- Fix overly aggressive cross-connection filter hiding legitimate
  multipoint wires in component diagrams

New Features:
- Add --2d flag to generate 2D diagrams (FS/BL only) instead of
  default 3D projection with WL axis
- Add component value and description to component diagram titles
  (e.g., "CB1: 30A - Circuit Breaker")

Enhancements:
- Update DEFAULT_WL_SCALE from 3.0 to 1.5 for better 3D projection
- Update diagram tests for independent X/Y scaling (scale_x, scale_y)
- Update wire label position to return axis name ('BL', 'FS', 'WL')

Test Updates:
- All 265 tests passing
- Update test fixtures (test_03, test_08)
- Add test_09_fixture for additional test coverage
- Remove obsolete test_07_fixture.csv

File Cleanup:
- Archive parser_netlist_ARCHIVED.py to docs/archive/

🤖 Generated with [Claude Code](https://claude.com/claude-code)

Co-Authored-By: Claude <noreply@anthropic.com>
Parts:
- L1: value (none) -> ~
Connections:
- net GND2 is gone; now on net GND1: BT1.2 (-), RG1.1 (GND)
- net GND3 is gone; now on net GND1: L1.2 (Out), L2.2 (Out), L3.2 (Out), LRU1.2 (Blk), SW1.1 (ON)
- net at FH1.Val_A (Desc): now also SW2.2 (IN)
