File: tests/fixtures/test_07_fixture.kicad_sch (KiCad schematic)
At the start: 7 parts, among them SW1 Desc, SW2 Desc

Commit message: code review by Claude. made few changes to test_07_fixture to address missing comments
Parts:
- BT1: LocLoad (0,0,0)S40 -> (10,0,0)S40
- FH1: LocLoad (none) -> (5,10,-4)R20
Changed lines of the file:
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@@
 			)
 		)
-		(property "LocLoad" "(0,0,0)S40"
+		(property "LocLoad" "(10,0,0)S40"
 			(at 151.13 109.22 0)
 			(effects
@@
 			(effects
 				(font
+					(size 1.27 1.27)
+				)
+				(hide yes)
+			)
+		)
+		(property "LocLoad" "(5,10,-4)R20"
+			(at 172.72 90.17 90)
+			(effects
+				(font

Commit message: updated test_07_fixture to have more realistic values"
Parts:
- BT1: LocLoad (10,0,0)S40 -> (30,5,0)S40
- L1: LocLoad (10,1,0)L10 -> (100,60,0)L10
- SW1: LocLoad (5,0,-1)R20 -> (5,10,-1)R20
- SW2: LocLoad (5,0,1)R20 -> (5,10,1)R20
Changed lines of the file:
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@@
 			)
 		)
-		(property "LocLoad" "(5,0,1)R20"
+		(property "LocLoad" "(5,10,1)R20"
 			(at 177.8 67.31 0)
 			(effects
@@
 			)
 		)
-		(property "LocLoad" "(10,0,0)S40"
+		(property "LocLoad" "(30,5,0)S40"
 			(at 151.13 109.22 0)
 			(effects
@@
 			)
 		)
-		(property "LocLoad" "(5,0,-1)R20"
+		(property "LocLoad" "(5,10,-1)R20"
 			(at 140.97 71.12 0)
 			(effects
@@
 			)
 		)
-		(property "Field5" ""
-			(at 175.26 49.53 0)
-			(effects
-				(font
-					(size 1.27 1.27)
-				)
-				(hide yes)
-			)
-		)
 		(property "LocLoad" "(10,0,-100)L7"
 			(at 175.26 49.53 0)
@@
 			)
 		)
-		(property "LocLoad" "(10,1,0)L10"
+		(property "LocLoad" "(100,60,0)L10"
 			(at 113.03 49.53 0)
 			(effects
